Commit message: Improve trot gait logic and smooth out stand-to-walk transitions

File: microspot_description/urdf/microspot.urdf (robot description, URDF)
Before this commit: robot my_robot, 18 links, 17 joints
Links:
- link base_link: mass 0.1 -> 0.5

Commit message: Create a 6 DoF arm and implement a controller for it

File: microspot_description/urdf/microspot.urdf (robot description, URDF)
Before this commit: robot my_robot, 18 links, 17 joints
Joints:
- removed joint base
- added joint base_joint: type fixed, parent world_link, child base_link, origin xyz=0 0 0.1 rpy=0 0 0
