Commit message: Improve URDF to simulate real robot and adapt controller to it

File: microspot_description/urdf/robot.urdf (robot description, URDF)
Before this commit: robot robot, 19 links, 18 joints
Joints:
- joint joint_1: axis -1.401298464324817e-45 -1.0 1.9721522630525295e-31 -> -1.401298464324817e-45 1.0 1.9721522630525295e-31; limit lower=0.0 upper=3.141593 effort=1000000 velocity=1000000 -> lower=-1.57 upper=1.57 effort=1000000 velocity=1000000

File: microspot_description/urdf/spot_arm.urdf.xacro (robot description, xacro)
@@ -1,10 +1,10 @@
 <?xml version="1.0"?>
 <robot name="spot_arm" xmlns:xacro="http://ros.org/wiki/xacro">
-    <xacro:include filename="$(find microspot_description)/urdf/microspot.urdf" />
+    <xacro:include filename="$(find microspot_description)/urdf/micro_v2.urdf" />
     <xacro:include filename="$(find microspot_description)/urdf/robot.urdf" />
     <joint name="microspot_to_arm_mount" type="fixed">
         <parent link="base_link"/>
         <child link="base_arm"/>
-        <origin xyz="0.05 0.0 0.03" rpy="0 3.14 0"/>
+        <origin xyz="0.05 0.0 0.03" rpy="1.57 0 0"/>
     </joint>
 </robot>
