Commit message: Fix controller node

File: microspot_description/urdf/micro_v2.urdf (robot description, URDF)
Before this commit: robot micro_v2, 41 links, 40 joints
Links:
- removed link front_right_end_foot_dummy_1
- added link back_left_thigh, mass 9.864601226263686e-07; collision mesh filename=package://microspot_description/meshes/back_left_thigh.stl scale=0.001 0.001 0.001; visual mesh filename=package://microspot_description/meshes/back_left_thigh.stl scale=0.001 0.001 0.001
- added link back_left_thigh_dummy, mass 9.864601226263686e-07; collision mesh filename=package://microspot_description/meshes/back_left_thigh_dumm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 scale=0.001 0.001 0.001; visual mesh filename=package://microspot_description/meshes/back_left_thigh_dumm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 scale=0.001 0.001 0.001
- added link back_right_thigh, mass 9.864601226263686e-07; collision mesh filename=package://microspot_description/meshes/back_right_thigh.stl scale=0.001 0.001 0.001; visual mesh filename=package://microspot_description/meshes/back_right_thigh.stl scale=0.001 0.001 0.001
- added link back_right_thigh_dummy, mass 9.864601226263686e-07; collision mesh filename=package://microspot_description/meshes/back_right_thigh_dum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 scale=0.001 0.001 0.001; visual mesh filename=package://microspot_description/meshes/back_right_thigh_dum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 scale=0.001 0.001 0.001
- added link front_left_thigh, mass 9.864601226263686e-07; collision mesh filename=package://microspot_description/meshes/front_left_thigh.stl scale=0.001 0.001 0.001; visual mesh filename=package://microspot_description/meshes/front_left_thigh.stl scale=0.001 0.001 0.001
- added link front_left_thigh_dummy, mass 9.864601226263686e-07; collision mesh filename=package://microspot_description/meshes/front_left_thigh_dum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 scale=0.001 0.001 0.001; visual mesh filename=package://microspot_description/meshes/front_left_thigh_dum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 scale=0.001 0.001 0.001
- added link front_right_thigh, mass 9.864601226263686e-07; collision mesh filename=package://microspot_description/meshes/front_right_thigh.stl scale=0.001 0.001 0.001; visual mesh filename=package://microspot_description/meshes/front_right_thigh.stl scale=0.001 0.001 0.001
- added link front_right_thigh_dummy, mass 9.864601226263686e-07; collision mesh filename=package://microspot_description/meshes/front_right_thigh_du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 scale=0.001 0.001 0.001; visual mesh filename=package://microspot_description/meshes/front_right_thigh_du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 scale=0.001 0.001 0.001
- link back_right_end_foot: mass 9.864601226263686e-07 -> 2.7304307462749233e-06; geometry collision mesh filename=package://microspot_description/meshes/back_right_foot_end.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 scale=0.001 0.001 0.001; visual mesh filename=package://microspot_description/meshes/back_right_foot_end.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 scale=0.001 0.001 0.001
- link back_right_end_foot_dummy: mass 9.864601226263686e-07 -> 6.165375766413709e-07
Joints:
- removed joint back_left_end_foot_dummy_Rigid-86
- removed joint back_right_end_foot_dummy_Rigid-87
- removed joint front_left_end_foot_dummy_Rigid-88
- removed joint front_right_end_foot_dummy_Rigid-85
- removed joint front_right_end_foot_dummy_joint
- added joint back_left_end_foot_dummy_Rigid-92: type fixed, parent back_left_end_foot_dummy, child back_left_end_foot, origin xyz=0.0 0.0 -0.24398324 rpy=1.734723475976807e-18 2.465190328815662e-32 -7.395570986446986e-31
- added joint back_left_thigh_Rigid-91: type fixed, parent back_left_thigh, child back_left_end_foot_dummy, origin xyz=0.0 -9.999999999994458e-06 -1.0999999999983245e-07 rpy=0.0 -0.0 1.8429380867263212e-47
- added joint back_left_thigh_dummy_Rigid-86: type fixed, parent back_left_thigh_dummy, child back_left_thigh, origin xyz=-0.00022351999999999927 0.018998680000000007 -0.012000000000000002 rpy=3.141592653589793 -1.5707963267948966 0
- added joint back_right_end_foot_dummy_Rigid-90: type fixed, parent back_right_end_foot_dummy, child back_right_end_foot, origin xyz=0.0 0.0 -0.244 rpy=0.0 5.254869241218064e-46 0.0
- added joint back_right_thigh_Rigid-89: type fixed, parent back_right_thigh, child back_right_end_foot_dummy, origin xyz=0.0 0.0 0.0 rpy=0.0 -0.0 0.0
- added joint back_right_thigh_dummy_Rigid-87: type fixed, parent back_right_thigh_dummy, child back_right_thigh, origin xyz=0.0 0.019000000000000003 0.011999999999999993 rpy=7.888609052210118e-31 1.5707963267948966 0
- added joint front_left_end_foot_dummy_Rigid-96: type fixed, parent front_left_end_foot_dummy, child front_left_end_foot, origin xyz=0.0 0.0 -0.24400000000000002 rpy=0.0 -0.0 0.0
- added joint front_left_thigh_dummy_Rigid-88: type fixed, parent front_left_thigh_dummy, child front_left_thigh, origin xyz=0.0 0.019000000000000003 -0.011999999999999993 rpy=3.141592653589793 -1.5707963267948966 0
- added joint front_left_thigh_dummy_Rigid-95: type fixed, parent front_left_thigh_dummy, child front_left_end_foot_dummy, origin xyz=0.0 0.019000000000000003 -0.011999999999999993 rpy=3.141592653589793 -1.5707963267948966 0
- added joint front_right_end_foot_dummy_Rigid-94: type fixed, parent front_right_end_foot_dummy, child front_right_end_foot, origin xyz=0.0 0.0 -0.244 rpy=0.0 -0.0 0.0
- added joint front_right_thigh_dummy_Rigid-85: type fixed, parent front_right_thigh_dummy, child front_right_thigh, origin xyz=-1.1102230246251566e-18 -0.018999999999999986 -0.01200000000000001 rpy=-3.141592653589793 -1.5707963267948966 0
- added joint front_right_thigh_dummy_Rigid-93: type fixed, parent front_right_thigh_dummy, child front_right_end_foot_dummy, origin xyz=-1.1102230246251566e-18 -0.018999999999999986 -0.01200000000000001 rpy=-3.141592653589793 -1.5707963267948966 0
- joint BL_hip_Rigid-84: child back_left_end_foot_dummy -> back_left_thigh_dummy; origin xyz=0.02424988000000001 -0.010749789999999999 0.02749999 rpy=1.5707963267948966 -3.0044506389506065e-32 1.5707963267948966 -> xyz=0.02424988000000001 -0.011072549999999999 0.027371629999999997 rpy=1.5707963267948966 -2.27259732694759e-31 1.5707963267948966
- joint BR_hip_Rigid-81: child back_right_end_foot_dummy -> back_right_thigh_dummy
- joint FL_hip_Rigid-82: child front_left_end_foot_dummy -> front_left_thigh_dummy
- joint FR_hip_Rigid-83: child front_right_end_foot_dummy_1 -> front_right_thigh_dummy
- joint back_left_hip_joint: axis 1.0 -7.174648137343064e-43 2.5243548967072624e-29 -> -1.0 -7.174648137343064e-43 2.5243548967072624e-29
- joint front_right_hip_joint: axis -1.0 1.9721522630525295e-31 -1.0088794678863922e-28 -> 1.0 1.9721522630525295e-31 -1.0088794678863922e-28
