Commit message: Fix some issues

File: spotmicro_description/urdf/micro_v2.urdf (robot description, URDF)
Before this commit: robot micro_v2, 48 links, 47 joints
Links:
- link BL_thigh_cover: geometry collision mesh filename=package://spotmicro_description/meshes/BL_thigh_cover.stl scale=0.001 0.001 0.001; visual mesh filename=package://spotmicro_description/meshes/BL_thigh_cover.stl scale=0.001 0.001 0.001
- link BR_thigh_cover: geometry collision mesh filename=package://spotmicro_description/meshes/BR_thigh_cover.stl scale=0.001 0.001 0.001; visual mesh filename=package://spotmicro_description/meshes/BR_thigh_cover.stl scale=0.001 0.001 0.001
- link B_I_shoulder: geometry collision mesh filename=package://spotmicro_description/meshes/B_I_shoulder.stl scale=0.001 0.001 0.001; visual mesh filename=package://spotmicro_description/meshes/B_I_shoulder.stl scale=0.001 0.001 0.001
- link B_O_shoulder: geometry collision mesh filename=package://spotmicro_description/meshes/B_O_shoulder.stl scale=0.001 0.001 0.001; visual mesh filename=package://spotmicro_description/meshes/B_O_shoulder.stl scale=0.001 0.001 0.001
- link B_cover: geometry collision mesh filename=package://spotmicro_description/meshes/B_cover.stl scale=0.001 0.001 0.001; visual mesh filename=package://spotmicro_description/meshes/B_cover.stl scale=0.001 0.001 0.001
- link FL_thigh_cover: geometry collision mesh filename=package://spotmicro_description/meshes/FL_thigh_cover.stl scale=0.001 0.001 0.001; visual mesh filename=package://spotmicro_description/meshes/FL_thigh_cover.stl scale=0.001 0.001 0.001
- link FR_thigh_cover: geometry collision mesh filename=package://spotmicro_description/meshes/FR_thigh_cover.stl scale=0.001 0.001 0.001; visual mesh filename=package://spotmicro_description/meshes/FR_thigh_cover.stl scale=0.001 0.001 0.001
- link F_I_shoulder: geometry collision mesh filename=package://spotmicro_description/meshes/F_I_shoulder.stl scale=0.001 0.001 0.001; visual mesh filename=package://spotmicro_description/meshes/F_I_shoulder.stl scale=0.001 0.001 0.001
- link F_O_shoulder: geometry collision mesh filename=package://spotmicro_description/meshes/F_O_shoulder.stl scale=0.001 0.001 0.001; visual mesh filename=package://spotmicro_description/meshes/F_O_shoulder.stl scale=0.001 0.001 0.001
- link F_cover: geometry collision mesh filename=package://spotmicro_description/meshes/F_cover.stl scale=0.001 0.001 0.001; visual mesh filename=package://spotmicro_description/meshes/F_cover.stl scale=0.001 0.001 0.001
- link L_side_plate: geometry collision mesh filename=package://spotmicro_description/meshes/L_side_plate.stl scale=0.001 0.001 0.001; visual mesh filename=package://spotmicro_description/meshes/L_side_plate.stl scale=0.001 0.001 0.001
- link R_side_plate: geometry collision mesh filename=package://spotmicro_description/meshes/R_side_plate.stl scale=0.001 0.001 0.001; visual mesh filename=package://spotmicro_description/meshes/R_side_plate.stl scale=0.001 0.001 0.001
- link T_cover: geometry collision mesh filename=package://spotmicro_description/meshes/T_cover.stl scale=0.001 0.001 0.001; visual mesh filename=package://spotmicro_description/meshes/T_cover.stl scale=0.001 0.001 0.001
- link back_left_end_foot: geometry collision mesh filename=package://spotmicro_description/meshes/back_left_end_foot.s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 scale=0.001 0.001 0.001; visual mesh filename=package://spotmicro_description/meshes/back_left_end_foot.s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 scale=0.001 0.001 0.001
- link back_left_end_foot_dummy: geometry collision mesh filename=package://spotmicro_description/meshes/back_left_end_foot_d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 scale=0.001 0.001 0.001; visual mesh filename=package://spotmicro_description/meshes/back_left_end_foot_d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 scale=0.001 0.001 0.001
- link back_left_foot_link: geometry collision mesh filename=package://spotmicro_description/meshes/BL_foot.stl scale=0.001 0.001 0.001; visual mesh filename=package://spotmicro_description/meshes/BL_foot.stl scale=0.001 0.001 0.001
- link back_left_hip_link: geometry collision mesh filename=package://spotmicro_description/meshes/BL_hip.stl scale=0.001 0.001 0.001; visual mesh filename=package://spotmicro_description/meshes/BL_hip.stl scale=0.001 0.001 0.001
- link back_left_knee_link: geometry collision mesh filename=package://spotmicro_description/meshes/BL_knee.stl scale=0.001 0.001 0.001; visual mesh filename=package://spotmicro_description/meshes/BL_knee.stl scale=0.001 0.001 0.001
- link back_left_thigh: geometry collision mesh filename=package://spotmicro_description/meshes/back_left_thigh.stl scale=0.001 0.001 0.001; visual mesh filename=package://spotmicro_description/meshes/back_left_thigh.stl scale=0.001 0.001 0.001
- link back_left_thigh_dummy: geometry collision mesh filename=package://spotmicro_description/meshes/back_left_thigh_dumm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 scale=0.001 0.001 0.001; visual mesh filename=package://spotmicro_description/meshes/back_left_thigh_dumm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 scale=0.001 0.001 0.001
- link back_left_thigh_link: geometry collision mesh filename=package://spotmicro_description/meshes/BL_thigh.stl scale=0.001 0.001 0.001; visual mesh filename=package://spotmicro_description/meshes/BL_thigh.stl scale=0.001 0.001 0.001
- link back_right_end_foot: geometry collision mesh filename=package://spotmicro_description/meshes/back_right_foot_end.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 scale=0.001 0.001 0.001; visual mesh filename=package://spotmicro_description/meshes/back_right_foot_end.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 scale=0.001 0.001 0.001
- link back_right_end_foot_dummy: geometry collision mesh filename=package://spotmicro_description/meshes/back_right_end_foot_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 scale=0.001 0.001 0.001; visual mesh filename=package://spotmicro_description/meshes/back_right_end_foot_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 scale=0.001 0.001 0.001
- link back_right_foot_link: geometry collision mesh filename=package://spotmicro_description/meshes/BR_foot.stl scale=0.001 0.001 0.001; visual mesh filename=package://spotmicro_description/meshes/BR_foot.stl scale=0.001 0.001 0.001
- link back_right_hip_link: geometry collision mesh filename=package://spotmicro_description/meshes/BR_hip.stl scale=0.001 0.001 0.001; visual mesh filename=package://spotmicro_description/meshes/BR_hip.stl scale=0.001 0.001 0.001
- link back_right_knee_link: geometry collision mesh filename=package://spotmicro_description/meshes/BR_knee.stl scale=0.001 0.001 0.001; visual mesh filename=package://spotmicro_description/meshes/BR_knee.stl scale=0.001 0.001 0.001
- link back_right_thigh: geometry collision mesh filename=package://spotmicro_description/meshes/back_right_thigh.stl scale=0.001 0.001 0.001; visual mesh filename=package://spotmicro_description/meshes/back_right_thigh.stl scale=0.001 0.001 0.001
- link back_right_thigh_dummy: geometry collision mesh filename=package://spotmicro_description/meshes/back_right_thigh_dum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 scale=0.001 0.001 0.001; visual mesh filename=package://spotmicro_description/meshes/back_right_thigh_dum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 scale=0.001 0.001 0.001
- link back_right_thigh_link: geometry collision mesh filename=package://spotmicro_description/meshes/BR_thigh.stl scale=0.001 0.001 0.001; visual mesh filename=package://spotmicro_description/meshes/BR_thigh.stl scale=0.001 0.001 0.001
- link base_link: geometry collision mesh filename=package://spotmicro_description/meshes/base_link.stl scale=0.001 0.001 0.001; visual mesh filename=package://spotmicro_description/meshes/base_link.stl scale=0.001 0.001 0.001
- link front_left_end_foot: geometry collision mesh filename=package://spotmicro_description/meshes/front_left_end_foot.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 scale=0.001 0.001 0.001; visual mesh filename=package://spotmicro_description/meshes/front_left_end_foot.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 scale=0.001 0.001 0.001
- link front_left_end_foot_dummy: geometry collision mesh filename=package://spotmicro_description/meshes/front_left_end_foot_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 scale=0.001 0.001 0.001; visual mesh filename=package://spotmicro_description/meshes/front_left_end_foot_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 scale=0.001 0.001 0.001
- link front_left_foot_link: geometry collision mesh filename=package://spotmicro_description/meshes/FL_foot.stl scale=0.001 0.001 0.001; visual mesh filename=package://spotmicro_description/meshes/FL_foot.stl scale=0.001 0.001 0.001
- link front_left_hip_link: geometry collision mesh filename=package://spotmicro_description/meshes/FL_hip.stl scale=0.001 0.001 0.001; visual mesh filename=package://spotmicro_description/meshes/FL_hip.stl scale=0.001 0.001 0.001
- link front_left_knee_link: geometry collision mesh filename=package://spotmicro_description/meshes/FL_knee.stl scale=0.001 0.001 0.001; visual mesh filename=package://spotmicro_description/meshes/FL_knee.stl scale=0.001 0.001 0.001
- link front_left_thigh: geometry collision mesh filename=package://spotmicro_description/meshes/front_left_thigh.stl scale=0.001 0.001 0.001; visual mesh filename=package://spotmicro_description/meshes/front_left_thigh.stl scale=0.001 0.001 0.001
- link front_left_thigh_dummy: geometry collision mesh filename=package://spotmicro_description/meshes/front_left_thigh_dum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 scale=0.001 0.001 0.001; visual mesh filename=package://spotmicro_description/meshes/front_left_thigh_dum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 scale=0.001 0.001 0.001
- link front_left_thigh_link: geometry collision mesh filename=package://spotmicro_description/meshes/FL_thigh.stl scale=0.001 0.001 0.001; visual mesh filename=package://spotmicro_description/meshes/FL_thigh.stl scale=0.001 0.001 0.001
- link front_right_end_foot: geometry collision mesh filename=package://spotmicro_description/meshes/front_right_end_foot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 scale=0.001 0.001 0.001; visual mesh filename=package://spotmicro_description/meshes/front_right_end_foot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 scale=0.001 0.001 0.001
- link front_right_end_foot_dummy: geometry collision mesh filename=package://spotmicro_description/meshes/front_right_end_foot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 scale=0.001 0.001 0.001; visual mesh filename=package://spotmicro_description/meshes/front_right_end_foot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 scale=0.001 0.001 0.001
- link front_right_foot_link: geometry collision mesh filename=package://spotmicro_description/meshes/FR_foot.stl scale=0.001 0.001 0.001; visual mesh filename=package://spotmicro_description/meshes/FR_foot.stl scale=0.001 0.001 0.001
- link front_right_hip_link: geometry collision mesh filename=package://spotmicro_description/meshes/FR_hip.stl scale=0.001 0.001 0.001; visual mesh filename=package://spotmicro_description/meshes/FR_hip.stl scale=0.001 0.001 0.001
- link front_right_knee_link: geometry collision mesh filename=package://spotmicro_description/meshes/FR_knee.stl scale=0.001 0.001 0.001; visual mesh filename=package://spotmicro_description/meshes/FR_knee.stl scale=0.001 0.001 0.001
- link front_right_thigh: geometry collision mesh filename=package://spotmicro_description/meshes/front_right_thigh.stl scale=0.001 0.001 0.001; visual mesh filename=package://spotmicro_description/meshes/front_right_thigh.stl scale=0.001 0.001 0.001
- link front_right_thigh_dummy: geometry collision mesh filename=package://spotmicro_description/meshes/front_right_thigh_du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 scale=0.001 0.001 0.001; visual mesh filename=package://spotmicro_description/meshes/front_right_thigh_du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 scale=0.001 0.001 0.001
- link front_right_thigh_link: geometry collision mesh filename=package://spotmicro_description/meshes/FR_thigh.stl scale=0.001 0.001 0.001; visual mesh filename=package://spotmicro_description/meshes/FR_thigh.stl scale=0.001 0.001 0.001
- link plate: geometry collision mesh filename=package://spotmicro_description/meshes/plate.stl scale=0.001 0.001 0.001; visual mesh filename=package://spotmicro_description/meshes/plate.stl scale=0.001 0.001 0.001

File: spotmicro_description/urdf/micro_v2_1.urdf (robot description, URDF)
Before this commit: robot micro_v2, 31 links, 30 joints
Links:
- link BL_thigh_cover: geometry collision mesh filename=package://spotmicro_description/meshes/BL_thigh_cover.stl scale=0.001 0.001 0.001; visual mesh filename=package://spotmicro_description/meshes/BL_thigh_cover.stl scale=0.001 0.001 0.001
- link BR_thigh_cover: geometry collision mesh filename=package://spotmicro_description/meshes/BR_thigh_cover.stl scale=0.001 0.001 0.001; visual mesh filename=package://spotmicro_description/meshes/BR_thigh_cover.stl scale=0.001 0.001 0.001
- link B_I_shoulder: geometry collision mesh filename=package://spotmicro_description/meshes/B_I_shoulder.stl scale=0.001 0.001 0.001; visual mesh filename=package://spotmicro_description/meshes/B_I_shoulder.stl scale=0.001 0.001 0.001
- link B_O_shoulder: geometry collision mesh filename=package://spotmicro_description/meshes/B_O_shoulder.stl scale=0.001 0.001 0.001; visual mesh filename=package://spotmicro_description/meshes/B_O_shoulder.stl scale=0.001 0.001 0.001
- link B_cover: geometry collision mesh filename=package://spotmicro_description/meshes/B_cover.stl scale=0.001 0.001 0.001; visual mesh filename=package://spotmicro_description/meshes/B_cover.stl scale=0.001 0.001 0.001
- link FL_thigh_cover: geometry collision mesh filename=package://spotmicro_description/meshes/FL_thigh_cover.stl scale=0.001 0.001 0.001; visual mesh filename=package://spotmicro_description/meshes/FL_thigh_cover.stl scale=0.001 0.001 0.001
- link FR_thigh_cover: geometry collision mesh filename=package://spotmicro_description/meshes/FR_thigh_cover.stl scale=0.001 0.001 0.001; visual mesh filename=package://spotmicro_description/meshes/FR_thigh_cover.stl scale=0.001 0.001 0.001
- link F_I_shoulder: geometry collision mesh filename=package://spotmicro_description/meshes/F_I_shoulder.stl scale=0.001 0.001 0.001; visual mesh filename=package://spotmicro_description/meshes/F_I_shoulder.stl scale=0.001 0.001 0.001
- link F_O_shoulder: geometry collision mesh filename=package://spotmicro_description/meshes/F_O_shoulder.stl scale=0.001 0.001 0.001; visual mesh filename=package://spotmicro_description/meshes/F_O_shoulder.stl scale=0.001 0.001 0.001
- link F_cover: geometry collision mesh filename=package://spotmicro_description/meshes/F_cover.stl scale=0.001 0.001 0.001; visual mesh filename=package://spotmicro_description/meshes/F_cover.stl scale=0.001 0.001 0.001
- link L_side_base_link: geometry collision mesh filename=package://spotmicro_description/meshes/L_side_plate.stl scale=0.001 0.001 0.001; visual mesh filename=package://spotmicro_description/meshes/L_side_plate.stl scale=0.001 0.001 0.001
- link R_side_base_link: geometry collision mesh filename=package://spotmicro_description/meshes/R_side_plate.stl scale=0.001 0.001 0.001; visual mesh filename=package://spotmicro_description/meshes/R_side_plate.stl scale=0.001 0.001 0.001
- link T_cover: geometry collision mesh filename=package://spotmicro_description/meshes/T_cover.stl scale=0.001 0.001 0.001; visual mesh filename=package://spotmicro_description/meshes/T_cover.stl scale=0.001 0.001 0.001
- link back_left_foot_link: geometry collision mesh filename=package://spotmicro_description/meshes/BL_foot.stl scale=0.001 0.001 0.001; visual mesh filename=package://spotmicro_description/meshes/BL_foot.stl scale=0.001 0.001 0.001
- link back_left_hip_link: geometry collision mesh filename=package://spotmicro_description/meshes/BL_hip.stl scale=0.001 0.001 0.001; visual mesh filename=package://spotmicro_description/meshes/BL_hip.stl scale=0.001 0.001 0.001
- link back_left_knee_link: geometry collision mesh filename=package://spotmicro_description/meshes/BL_knee.stl scale=0.001 0.001 0.001; visual mesh filename=package://spotmicro_description/meshes/BL_knee.stl scale=0.001 0.001 0.001
- link back_left_thigh_link: geometry collision mesh filename=package://spotmicro_description/meshes/BL_thigh.stl scale=0.001 0.001 0.001; visual mesh filename=package://spotmicro_description/meshes/BL_thigh.stl scale=0.001 0.001 0.001
- link back_right_foot_link: geometry collision mesh filename=package://spotmicro_description/meshes/BR_foot.stl scale=0.001 0.001 0.001; visual mesh filename=package://spotmicro_description/meshes/BR_foot.stl scale=0.001 0.001 0.001
- link back_right_hip_link: geometry collision mesh filename=package://spotmicro_description/meshes/BR_hip.stl scale=0.001 0.001 0.001; visual mesh filename=package://spotmicro_description/meshes/BR_hip.stl scale=0.001 0.001 0.001
- link back_right_knee_link: geometry collision mesh filename=package://spotmicro_description/meshes/BR_knee.stl scale=0.001 0.001 0.001; visual mesh filename=package://spotmicro_description/meshes/BR_knee.stl scale=0.001 0.001 0.001
- link back_right_thigh_link: geometry collision mesh filename=package://spotmicro_description/meshes/BR_thigh.stl scale=0.001 0.001 0.001; visual mesh filename=package://spotmicro_description/meshes/BR_thigh.stl scale=0.001 0.001 0.001
- link base_link: geometry collision mesh filename=package://spotmicro_description/meshes/plate.stl scale=0.001 0.001 0.001; visual mesh filename=package://spotmicro_description/meshes/plate.stl scale=0.001 0.001 0.001
- link front_left_foot_link: geometry collision mesh filename=package://spotmicro_description/meshes/FL_foot.stl scale=0.001 0.001 0.001; visual mesh filename=package://spotmicro_description/meshes/FL_foot.stl scale=0.001 0.001 0.001
- link front_left_hip_link: geometry collision mesh filename=package://spotmicro_description/meshes/FL_hip.stl scale=0.001 0.001 0.001; visual mesh filename=package://spotmicro_description/meshes/FL_hip.stl scale=0.001 0.001 0.001
- link front_left_knee_link: geometry collision mesh filename=package://spotmicro_description/meshes/FL_knee.stl scale=0.001 0.001 0.001; visual mesh filename=package://spotmicro_description/meshes/FL_knee.stl scale=0.001 0.001 0.001
- link front_left_thigh_link: geometry collision mesh filename=package://spotmicro_description/meshes/FL_thigh.stl scale=0.001 0.001 0.001; visual mesh filename=package://spotmicro_description/meshes/FL_thigh.stl scale=0.001 0.001 0.001
- link front_right_foot_link: geometry collision mesh filename=package://spotmicro_description/meshes/FR_foot.stl scale=0.001 0.001 0.001; visual mesh filename=package://spotmicro_description/meshes/FR_foot.stl scale=0.001 0.001 0.001
- link front_right_hip_link: geometry collision mesh filename=package://spotmicro_description/meshes/FR_hip.stl scale=0.001 0.001 0.001; visual mesh filename=package://spotmicro_description/meshes/FR_hip.stl scale=0.001 0.001 0.001
- link front_right_knee_link: geometry collision mesh filename=package://spotmicro_description/meshes/FR_knee.stl scale=0.001 0.001 0.001; visual mesh filename=package://spotmicro_description/meshes/FR_knee.stl scale=0.001 0.001 0.001
- link front_right_thigh_link: geometry collision mesh filename=package://spotmicro_description/meshes/FR_thigh.stl scale=0.001 0.001 0.001; visual mesh filename=package://spotmicro_description/meshes/FR_thigh.stl scale=0.001 0.001 0.001

File: spotmicro_description/urdf/robot.urdf (robot description, URDF)
Before this commit: robot robot, 19 links, 18 joints
Links:
- link base_arm: geometry collision mesh filename=package://spotmicro_description/meshes/base_arm.stl scale=0.001 0.001 0.001; visual mesh filename=package://spotmicro_description/meshes/base_arm.stl scale=0.001 0.001 0.001
- link gripper: geometry collision mesh filename=package://spotmicro_description/meshes/gripper.stl scale=0.001 0.001 0.001; visual mesh filename=package://spotmicro_description/meshes/gripper.stl scale=0.001 0.001 0.001
- link link_1: geometry collision mesh filename=package://spotmicro_description/meshes/link_1.stl scale=0.001 0.001 0.001; visual mesh filename=package://spotmicro_description/meshes/link_1.stl scale=0.001 0.001 0.001
- link link_10: geometry collision mesh filename=package://spotmicro_description/meshes/link_10.stl scale=0.001 0.001 0.001; visual mesh filename=package://spotmicro_description/meshes/link_10.stl scale=0.001 0.001 0.001
- link link_11: geometry collision mesh filename=package://spotmicro_description/meshes/link_11.stl scale=0.001 0.001 0.001; visual mesh filename=package://spotmicro_description/meshes/link_11.stl scale=0.001 0.001 0.001
- link link_2: geometry collision mesh filename=package://spotmicro_description/meshes/link_2.stl scale=0.001 0.001 0.001; visual mesh filename=package://spotmicro_description/meshes/link_2.stl scale=0.001 0.001 0.001
- link link_3: geometry collision mesh filename=package://spotmicro_description/meshes/link_3.stl scale=0.001 0.001 0.001; visual mesh filename=package://spotmicro_description/meshes/link_3.stl scale=0.001 0.001 0.001
- link link_4: geometry collision mesh filename=package://spotmicro_description/meshes/link_4.stl scale=0.001 0.001 0.001; visual mesh filename=package://spotmicro_description/meshes/link_4.stl scale=0.001 0.001 0.001
- link link_5: geometry collision mesh filename=package://spotmicro_description/meshes/link_5.stl scale=0.001 0.001 0.001; visual mesh filename=package://spotmicro_description/meshes/link_5.stl scale=0.001 0.001 0.001
- link link_6: geometry collision mesh filename=package://spotmicro_description/meshes/link_6.stl scale=0.001 0.001 0.001; visual mesh filename=package://spotmicro_description/meshes/link_6.stl scale=0.001 0.001 0.001
- link link_7: geometry collision mesh filename=package://spotmicro_description/meshes/link_7.stl scale=0.001 0.001 0.001; visual mesh filename=package://spotmicro_description/meshes/link_7.stl scale=0.001 0.001 0.001
- link link_8: geometry collision mesh filename=package://spotmicro_description/meshes/link_8.stl scale=0.001 0.001 0.001; visual mesh filename=package://spotmicro_description/meshes/link_8.stl scale=0.001 0.001 0.001
- link link_9: geometry collision mesh filename=package://spotmicro_description/meshes/link_9.stl scale=0.001 0.001 0.001; visual mesh filename=package://spotmicro_description/meshes/link_9.stl scale=0.001 0.001 0.001
- link rotor_1: geometry collision mesh filename=package://spotmicro_description/meshes/rotor_1.stl scale=0.001 0.001 0.001; visual mesh filename=package://spotmicro_description/meshes/rotor_1.stl scale=0.001 0.001 0.001
- link rotor_2: geometry collision mesh filename=package://spotmicro_description/meshes/rotor_2.stl scale=0.001 0.001 0.001; visual mesh filename=package://spotmicro_description/meshes/rotor_2.stl scale=0.001 0.001 0.001
- link rotor_3: geometry collision mesh filename=package://spotmicro_description/meshes/rotor_3.stl scale=0.001 0.001 0.001; visual mesh filename=package://spotmicro_description/meshes/rotor_3.stl scale=0.001 0.001 0.001
- link rotor_4: geometry collision mesh filename=package://spotmicro_description/meshes/rotor_4.stl scale=0.001 0.001 0.001; visual mesh filename=package://spotmicro_description/meshes/rotor_4.stl scale=0.001 0.001 0.001
- link rotor_5: geometry collision mesh filename=package://spotmicro_description/meshes/rotor_5.stl scale=0.001 0.001 0.001; visual mesh filename=package://spotmicro_description/meshes/rotor_5.stl scale=0.001 0.001 0.001
- link rotor_6: geometry collision mesh filename=package://spotmicro_description/meshes/rotor_6.stl scale=0.001 0.001 0.001; visual mesh filename=package://spotmicro_description/meshes/rotor_6.stl scale=0.001 0.001 0.001
