Commit message: Fix some issues

File: spotmicro_description/urdf/robot_arm.urdf (robot description, URDF)
Before this commit: robot robot_arm, 17 links, 16 joints
Links:
- link base: geometry collision mesh filename=package://spotmicro_description/meshes/base.stl scale=0.001 0.001 0.001; visual mesh filename=package://spotmicro_description/meshes/base.stl scale=0.001 0.001 0.001
- link link_1: geometry collision mesh filename=package://spotmicro_description/meshes/base_rotor.stl scale=0.001 0.001 0.001; visual mesh filename=package://spotmicro_description/meshes/base_rotor.stl scale=0.001 0.001 0.001
- link link_10: geometry collision mesh filename=package://spotmicro_description/meshes/drivesmall.stl scale=0.001 0.001 0.001; visual mesh filename=package://spotmicro_description/meshes/drivesmall.stl scale=0.001 0.001 0.001
- link link_11: geometry collision mesh filename=package://spotmicro_description/meshes/drivesmall_rotor-3.s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 scale=0.001 0.001 0.001; visual mesh filename=package://spotmicro_description/meshes/drivesmall_rotor-3.s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 scale=0.001 0.001 0.001
- link link_12: geometry collision mesh filename=package://spotmicro_description/meshes/drivesmall-2.stl scale=0.001 0.001 0.001; visual mesh filename=package://spotmicro_description/meshes/drivesmall-2.stl scale=0.001 0.001 0.001
- link link_13: geometry collision mesh filename=package://spotmicro_description/meshes/drivesmall_rotor-4.s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 scale=0.001 0.001 0.001; visual mesh filename=package://spotmicro_description/meshes/drivesmall_rotor-4.s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 scale=0.001 0.001 0.001
- link link_14: geometry collision mesh filename=package://spotmicro_description/meshes/drivesmall-1.stl scale=0.001 0.001 0.001; visual mesh filename=package://spotmicro_description/meshes/drivesmall-1.stl scale=0.001 0.001 0.001
- link link_15: geometry collision mesh filename=package://spotmicro_description/meshes/drivesmall_rotor.stl scale=0.001 0.001 0.001; visual mesh filename=package://spotmicro_description/meshes/drivesmall_rotor.stl scale=0.001 0.001 0.001
- link link_2: geometry collision mesh filename=package://spotmicro_description/meshes/drivebig.stl scale=0.001 0.001 0.001; visual mesh filename=package://spotmicro_description/meshes/drivebig.stl scale=0.001 0.001 0.001
- link link_3: geometry collision mesh filename=package://spotmicro_description/meshes/drivesmall_rotor-1.s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 scale=0.001 0.001 0.001; visual mesh filename=package://spotmicro_description/meshes/drivesmall_rotor-1.s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 scale=0.001 0.001 0.001
- link link_4: geometry collision mesh filename=package://spotmicro_description/meshes/connector_corner.stl scale=0.001 0.001 0.001; visual mesh filename=package://spotmicro_description/meshes/connector_corner.stl scale=0.001 0.001 0.001
- link link_5: geometry collision mesh filename=package://spotmicro_description/meshes/connector_straight.s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 scale=0.001 0.001 0.001; visual mesh filename=package://spotmicro_description/meshes/connector_straight.s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 scale=0.001 0.001 0.001
- link link_6: geometry collision mesh filename=package://spotmicro_description/meshes/drivebig-1.stl scale=0.001 0.001 0.001; visual mesh filename=package://spotmicro_description/meshes/drivebig-1.stl scale=0.001 0.001 0.001
- link link_7: geometry collision mesh filename=package://spotmicro_description/meshes/drivesmall_rotor-2.s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 scale=0.001 0.001 0.001; visual mesh filename=package://spotmicro_description/meshes/drivesmall_rotor-2.s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 scale=0.001 0.001 0.001
- link link_8: geometry collision mesh filename=package://spotmicro_description/meshes/connector_corner-1.s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 scale=0.001 0.001 0.001; visual mesh filename=package://spotmicro_description/meshes/connector_corner-1.s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 scale=0.001 0.001 0.001
- link link_9: geometry collision mesh filename=package://spotmicro_description/meshes/connector_straight-1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 scale=0.001 0.001 0.001; visual mesh filename=package://spotmicro_description/meshes/connector_straight-1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 scale=0.001 0.001 0.001
